File: design_files/ASD2005.brd (EAGLE design)
At the start: 34.6 x 31.6 mm, 6 parts, among them J1 DF12-32-DS, J2 ESDM12100, J3 ESDM09100, J4 ESDM09100, J6 DF12-32-DP

Commit message: updates format
Parts:
- moved U$1 12.0 mm to (55.9, 0.00)
- moved J1 8.60 mm to (25.0, 21.3)
- moved J2 8.60 mm to (25.0, 12.0)
- moved J3 8.60 mm to (39.0, 27.2)
- moved J4 8.60 mm to (11.0, 27.2)
- moved J6 8.60 mm to (25.0, 21.3)
Routing:
- net AD5/SCL: track 16.1 -> 13.7 mm
Other:
- board size 34.6 x 31.6 mm -> 34.6 x 30.3 mm
- board text added: "ASD2005 - Rev2"
- board text added: "RX"
- board text added: "SCL"
- board text added: "SDA"
- board text added: "TX"
- board text added: "TinyCircuits.com"
- board text added: "^ V-SCORE EDGE ALONG OUTLINE ^"
- board text removed: "ASD2005 - Rev1"
- board text removed: "Tiny-Circuits.com"
