File: design_files/ASD2005.sch (EAGLE design)
At the start: 5 parts, among them J1 DF12-32-DS, J2 ESDM12100, J3 ESDM09100, J4 ESDM09100, J6 DF12-32-DP

Commit message: updates format
Other:
- note added: "2"
- note removed: "1"
Changed lines of the file:
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@@
 <text x="340.868" y="17.272" size="2.54" layer="94" font="vector">TinyShield - Proto Terminals Board</text>
 <text x="327.152" y="6.35" size="3.556" layer="94" font="vector">AS-SCH-ASD2005</text>
-<text x="416.56" y="6.858" size="3.556" layer="94" font="vector">1</text>
+<text x="416.56" y="6.858" size="3.556" layer="94" font="vector">2</text>
 <text x="304.8" y="165.354" size="1.778" layer="91">IOREF</text>
 <text x="45.72" y="35.56" size="3.048" layer="91">Released under the Creative Commons Attribution Share-Alike 3.0 License</text>
